Commit message: my_robot

File: ros_ws/src/my_robot/urdf/my_robot.urdf (robot description, URDF)
Before this commit: robot my_robot, 10 links, 9 joints
Links:
- removed link base_footprint
- added link base_dummy
Joints:
- removed joint base_footprint_joint
- added joint base_dummy_joint: type fixed, parent base_dummy, child base_link, origin xyz=0 0 0 rpy=0 0 0
