Commit message: editing name

File: ros_ws/src/my_robot/urdf/sensors.xacro (robot description, xacro)
@@ -3,5 +3,5 @@
     <joint name="lidar_joint" type="fixed">
         <parent link="base_link"/>
-        <child link="lidar_link"/>
+        <child link="lidar_frame"/>
         <origin xyz = "0.3 0 0.4"/>
     </joint>

Commit message: Fixing dimensions

File: ros_ws/src/my_robot/urdf/sensors.xacro (robot description, xacro)
@@ -4,5 +4,5 @@
         <parent link="base_link"/>
         <child link="lidar_frame"/>
-        <origin xyz = "0.3 0 0.4"/>
+        <origin xyz = "0.3 0 0.29"/>
     </joint>
     <link name="lidar_frame">

Commit message: Fixing bugs

File: ros_ws/src/my_robot/urdf/sensors.xacro (robot description, xacro)
@@ -20,8 +20,8 @@
         <inertial>
             	<mass value="1.0"/>
-        		<!-- Cylinder: r=0.15, h=0.08, mass=1.0 -->
-        		<!-- ixx = (1/12)*1*(3*0.15^2 + 0.08^2) = 0.006 -->
-        		<!-- iyy = (1/12)*1*(3*0.15^2 + 0.08^2) = 0.006 -->
-        		<!-- izz = (1/2)*1*0.15^2 = 0.011 -->
+            	<!-- Cylinder: r=0.15, h=0.08, mass=1.0 -->
+            	<!-- ixx = (1/12)*1*(3*0.15^2 + 0.08^2) = 0.006 -->
+            	<!-- iyy = (1/12)*1*(3*0.15^2 + 0.08^2) = 0.006 -->
+            	<!-- izz = (1/2)*1*0.15^2 = 0.011 -->
             	<inertia
             		ixx="0.006" ixy="0.0" ixz="0.0"
@@ -29,6 +29,4 @@
             		izz="0.011"/>
         </inertial>
-    </link>
-    <gazebo reference="lidar_frame">
         <sensor name="lidar_sensor" type="lidar">
             <pose>0 0 0 0 0 0</pose>
@@ -51,4 +49,4 @@
             </lidar>
         </sensor>
-    </gazebo>
+    </link>
 </robot>

Commit message: Fixing Bugs

File: ros_ws/src/my_robot/urdf/sensors.xacro (robot description, xacro)
@@ -29,4 +29,6 @@
             		izz="0.011"/>
         </inertial>
+    </link>
+    <gazebo reference="lidar_frame">
         <sensor name="lidar_sensor" type="gpu_lidar">
             <pose>0 0 0 0 0 0</pose>
@@ -49,4 +51,4 @@
             </lidar>
         </sensor>
-    </link>
+    </gazebo>
 </robot>

Commit message: Imu

File: ros_ws/src/my_robot/urdf/sensors.xacro (robot description, xacro)
@@ -30,4 +30,17 @@
         </inertial>
     </link>
+    <link name="imu_link">
+        <inertial>
+            <mass value="0.01"/>
+            <inertia ixx="0.001" ixy="0.0" ixz="0.0"
+                     iyy="0.001" iyz="0.0"
+                     izz="0.001"/>
+        </inertial>
+    </link>
+    <joint name="imu_joint" type="fixed">
+        <parent link="base_link"/>
+        <child link="imu_link"/>
+        <origin xyz = "0 0 0"/>
+    </joint>
     <gazebo reference="lidar_frame">
         <sensor name="lidar_sensor" type="gpu_lidar">
@@ -55,3 +68,19 @@
         </sensor>
     </gazebo>
+    <gazebo reference="imu_link">
+        <sensor name="imu_sensor" type="imu">
+            <always_on>1</always_on>
+            <update_rate>10</update_rate>
+            <visual>true</visual>
+            <topic>/imu/data</topic>
+            <ignition_frame_id>imu_link</ignition_frame_id>
+            <plugin name="imu_plugin" filename="libgazebo_ros_imu_sensor.so">
+                <ros>
+                    <namespace>/imu</namespace>
+                    <topic>~/out:=data</topic>
+                </ros>
+                <initial_orientation_as_reference>false</initial_orientation_as_reference>
+            </plugin>
+        </sensor>
+    </gazebo>
 </robot>

Commit message: Imu

File: ros_ws/src/my_robot/urdf/sensors.xacro (robot description, xacro)
@@ -72,13 +72,9 @@
             <always_on>1</always_on>
             <update_rate>10</update_rate>
-            <visual>true</visual>
+            <visualize>true</visualize>
             <topic>/imu/data</topic>
             <ignition_frame_id>imu_link</ignition_frame_id>
-            <plugin name="imu_plugin" filename="libgazebo_ros_imu_sensor.so">
-                <ros>
-                    <namespace>/imu</namespace>
-                    <topic>~/out:=data</topic>
-                </ros>
-                <initial_orientation_as_reference>false</initial_orientation_as_reference>
+            <plugin filename="libignition-gazebo-imu-system.so"
+                    name="ignition::gazebo::systems::Imu">
             </plugin>
         </sensor>

Commit message: Fixing Lidar

File: ros_ws/src/my_robot/urdf/sensors.xacro (robot description, xacro)
@@ -4,5 +4,5 @@
         <parent link="base_link"/>
         <child link="lidar_frame"/>
-        <origin xyz = "0.3 0 0.29"/>
+        <origin xyz = "0.3 0 -0.29"/>
     </joint>
     <link name="lidar_frame">
@@ -61,5 +61,5 @@
                 </scan>
                 <range>
-                    <min>0.3</min>
+                    <min>1</min>
                     <max>10</max>
                     <resolution>0.01</resolution>

Commit message: Fixing Lidar

File: ros_ws/src/my_robot/urdf/sensors.xacro (robot description, xacro)
@@ -4,5 +4,5 @@
         <parent link="base_link"/>
         <child link="lidar_frame"/>
-        <origin xyz = "0.3 0 -0.29"/>
+        <origin xyz = "0 0 -0.29"/>
     </joint>
     <link name="lidar_frame">
