Commit message: Adding an arm

File: ros_ws/src/my_robot/urdf/arm.xacro (robot description, xacro)
@@ -34,5 +34,5 @@
         <child link="arm_link"/>
         <origin xyz="0 0 0.04"/>
-        <axis xyz = "0 0 1"/>
+        <axis xyz = "0 1 0"/>
         <limit lower="-1.57" upper="1.57" effort="1000" velocity="1"/>
     </joint>
@@ -42,5 +42,5 @@
                 <box size="0.1 0.1 0.5"/>
             </geometry>
-            <origin xyz = "0 0 0"/>
+            <origin xyz = "0 0 -0.21"/>
             <material name = "black"/>
         </visual>

Commit message: Adding an arm

File: ros_ws/src/my_robot/urdf/arm.xacro (robot description, xacro)
@@ -42,5 +42,5 @@
                 <box size="0.1 0.1 0.5"/>
             </geometry>
-            <origin xyz = "0 0 -0.21"/>
+            <origin xyz = "0 0 0.21"/>
             <material name = "black"/>
         </visual>

Commit message: Updating arm

File: ros_ws/src/my_robot/urdf/arm.xacro (robot description, xacro)
@@ -4,5 +4,5 @@
         <parent link="base_link"/>
         <child link="arm_base"/>
-        <origin xyz="-0.3 0 0.29"/>
+        <origin xyz="0.3 0 0.29"/>
     </joint>
     <link name="arm_base">
@@ -47,16 +47,16 @@
         <collision>
             <geometry>
-                <box size="0.1 0.1 0.5"/>
+                <box size="0.1 0.1 1"/>
             </geometry>
         </collision>
         <inertial>
             <mass value="1.0"/>
-            <!-- Box: 0.1 x 0.1 x 0.5, mass=1.0 -->
-            <!-- ixx = (1/12)*1*(0.1^2 + 0.5^2) = 0.022 -->
-            <!-- iyy = (1/12)*1*(0.1^2 + 0.5^2) = 0.022 -->
+            <!-- Box: 0.1 x 0.1 x 1, mass=1.0 -->
+            <!-- ixx = (1/12)*1*(0.1^2 + 1^2) = 0.084 -->
+            <!-- iyy = (1/12)*1*(0.1^2 + 1^2) = 0.084 -->
             <!-- izz = (1/12)*1*(0.1^2 + 0.1^2) = 0.0017 -->
             <inertia
-                ixx="0.022" ixy="0.0" ixz="0.0"
-                iyy="0.022" iyz="0.0"
+                ixx="0.084" ixy="0.0" ixz="0.0"
+                iyy="0.084" iyz="0.0"
                 izz="0.0017"/>
         </inertial>

Commit message: Updating arm

File: ros_ws/src/my_robot/urdf/arm.xacro (robot description, xacro)
@@ -40,7 +40,7 @@
         <visual>
             <geometry>
-                <box size="0.1 0.1 0.5"/>
+                <box size="0.1 0.1 1"/>
             </geometry>
-            <origin xyz = "0 0 0.21"/>
+            <origin xyz = "0 0 0.71"/>
             <material name = "black"/>
         </visual>

Commit message: Updating arm

File: ros_ws/src/my_robot/urdf/arm.xacro (robot description, xacro)
@@ -42,5 +42,5 @@
                 <box size="0.1 0.1 1"/>
             </geometry>
-            <origin xyz = "0 0 0.71"/>
+            <origin xyz = "0 0 0.46"/>
             <material name = "black"/>
         </visual>

Commit message: Updating arm

File: ros_ws/src/my_robot/urdf/arm.xacro (robot description, xacro)
@@ -4,5 +4,5 @@
         <parent link="base_link"/>
         <child link="arm_base"/>
-        <origin xyz="0.3 0 0.29"/>
+        <origin xyz="0 0 0.29"/>
     </joint>
     <link name="arm_base">

Commit message: Fixing camera to arm

File: ros_ws/src/my_robot/urdf/arm.xacro (robot description, xacro)
@@ -49,4 +49,5 @@
                 <box size="0.1 0.1 1"/>
             </geometry>
+            <origin xyz = "0 0 0.46"/>
         </collision>
         <inertial>

File: ros_ws/src/my_robot/urdf/camera.xacro (robot description, xacro)
@@ -4,5 +4,5 @@
         <parent link="arm_link"/>
         <child link="camera_frame"/>
-        <origin xyz = "0 0 0.101"/>
+        <origin xyz = "0 0 1.01"/>
     </joint>
     <link name="camera_frame">

Commit message: adding rqt_joint_trajectory_controller

File: ros_ws/src/my_robot/urdf/arm.xacro (robot description, xacro)
@@ -1,4 +1,4 @@
 <?xml version="1.0"?>
-<robot xmlns:xacro="http://www.ros.org/wiki/xacro" name="panda">
+<robot xmlns:xacro="http://www.ros.org/wiki/xacro">
     <joint name="arm_base_joint" type="fixed">
         <parent link="base_link"/>
@@ -63,3 +63,21 @@
         </inertial>
     </link>
+    <ros2_control name="IgnitionSystem" type="system">
+        <hardware>
+            <plugin>ign_ros2_control/IgnitionSystem</plugin>
+        </hardware>
+        <joint name="arm_joint">
+            <command_interface name="position">
+                <param name="min">-1.57</param>
+                <param name="max">1.57</param>
+            </command_interface>
+            <state_interface name="position"/>
+            <state_interface name="velocity"/>
+        </joint>
+    </ros2_control>
+    <gazebo>
+        <plugin filename="ign_ros2_control-system" name="ign_ros2_control::IgnitionROS2ControlSystem">
+            <parameters>$(find my_robot)/config/controllers.yaml</parameters>
+        </plugin>
+    </gazebo>
 </robot>
