Commit message: Camera_optical

File: ros_ws/src/my_robot/urdf/camera.xacro (robot description, xacro)
@@ -9,5 +9,5 @@
         <visual>
 			<geometry>
-				<cylinder radius = "0.02" length = "0.01"/>
+				<cylinder radius = "0.05" length = "0.01"/>
 			</geometry>
 			<material name="red"/>
@@ -15,4 +15,10 @@
 		</visual>
     </link>
+    <joint name="camera_optical_joint" type="fixed">
+        <parent link="camera_frame"/>
+        <child link="camera_optical_frame"/>
+        <origin xyz = "0 0 0" rpy="${-pi/2} 0 ${-pi/2}"/>
+    </joint>
+    <link name="camera_optical_frame"/>
     <gazebo reference="camera_frame">
         <!-- <sensor name="camera_sensor" type="gpu_lidar">

Commit message: Fixing camera to arm

File: ros_ws/src/my_robot/urdf/camera.xacro (robot description, xacro)
@@ -2,7 +2,7 @@
 <robot xmlns:xacro="http://www.ros.org/wiki/xacro">
     <joint name="camera_joint" type="fixed">
-        <parent link="base_link"/>
+        <parent link="arm_link"/>
         <child link="camera_frame"/>
-        <origin xyz = "0.905 0 0.1"/>
+        <origin xyz = "0 0 0.55"/>
     </joint>
     <link name="camera_frame">

Commit message: Fixing camera to arm

File: ros_ws/src/my_robot/urdf/camera.xacro (robot description, xacro)
@@ -4,5 +4,5 @@
         <parent link="arm_link"/>
         <child link="camera_frame"/>
-        <origin xyz = "0 0 0.55"/>
+        <origin xyz = "0 0 0.101"/>
     </joint>
     <link name="camera_frame">
@@ -12,5 +12,5 @@
 			</geometry>
 			<material name="red"/>
-            <origin rpy = "0 1.5708 0"/>
+            <origin rpy = "0 0 0"/>
 		</visual>
     </link>

Commit message: Fixing camera to arm

File: ros_ws/src/my_robot/urdf/camera.xacro (robot description, xacro)
@@ -4,5 +4,5 @@
         <parent link="arm_link"/>
         <child link="camera_frame"/>
-        <origin xyz = "0 0 1.01"/>
+        <origin xyz = "0 0 0.96"/>
     </joint>
     <link name="camera_frame">

Commit message: Fixing

File: ros_ws/src/my_robot/urdf/camera.xacro (robot description, xacro)
@@ -4,5 +4,5 @@
         <parent link="arm_link"/>
         <child link="camera_frame"/>
-        <origin xyz = "0 0 0.96"/>
+        <origin xyz="0 0 0.96" rpy="0 ${-pi/2} 0"/>
     </joint>
     <link name="camera_frame">

Commit message: Fixing

File: ros_ws/src/my_robot/urdf/camera.xacro (robot description, xacro)
@@ -4,5 +4,5 @@
         <parent link="arm_link"/>
         <child link="camera_frame"/>
-        <origin xyz="0 0 0.96" rpy="0 ${-pi/2} 0"/>
+        <origin xyz="0 0 0.96" rpy="0 0 0"/>
     </joint>
     <link name="camera_frame">
@@ -18,10 +18,10 @@
         <parent link="camera_frame"/>
         <child link="camera_optical_frame"/>
-        <origin xyz = "0 0 0" rpy="${-pi/2} 0 ${-pi/2}"/>
+        <origin xyz="0 0 0" rpy="0 0 ${-pi/2}"/>
     </joint>
     <link name="camera_optical_frame"/>
     <gazebo reference="camera_frame">
         <sensor name="camera_sensor" type="camera">
-            <pose>0 0 0 0 0 0</pose>
+            <pose>0 0 0 0 -1.57079632679 0</pose>
             <visualize>true</visualize>
             <update_rate>10</update_rate>
